Commit message: dfirst prototype

File: src/the_8th_leg_description/urdf/the_8th_leg.urdf (robot description, URDF)
Before this commit: robot the_8th_leg, 3 links, 2 joints
Links:
- added link link_3, mass 1.0; collision cylinder length=0.2 radius=0.04; visual cylinder length=0.2 radius=0.04
- added link link_4, mass 1.0; collision cylinder length=0.2 radius=0.035; visual cylinder length=0.2 radius=0.035
- added link link_5, mass 1.0; collision cylinder length=0.05 radius=0.03; visual cylinder length=0.05 radius=0.03
- added link link_6, mass 1.0; collision cylinder length=0.04 radius=0.03; visual cylinder length=0.04 radius=0.03
- added link link_7, mass 1.0; collision cylinder length=0.04 radius=0.025; visual cylinder length=0.04 radius=0.025
- link link_2: geometry collision cylinder length=0.09 radius=0.05; visual cylinder length=0.09 radius=0.05
Joints:
- added joint base_to_shoulder: type revolute, parent link_2, child link_3, origin xyz=0 0 0.09, axis 0 1 0, limit lower=-1.88496 upper=1.98968 effort=10.0 velocity=1.0
- added joint elbow_to_wrist_pitch: type revolute, parent link_4, child link_5, origin xyz=0 0 0.2, axis 0 1 0, limit lower=-1.74533 upper=2.14675 effort=10.0 velocity=1.0
- added joint shoulder_to_elbow: type revolute, parent link_3, child link_4, origin xyz=0 0 0.2, axis 0 1 0, limit lower=-0.57596 upper=2.61799 effort=10.0 velocity=1.0
- added joint wrist_pitch_to_roll: type revolute, parent link_5, child link_6, origin xyz=0 0 0.05, axis 0 0 1, limit lower=-3.14159 upper=3.14159 effort=10.0 velocity=1.0
- added joint wrist_roll_to_yaw: type revolute, parent link_6, child link_7, origin xyz=0 0 0.04, axis 1 0 0, limit lower=-1.57080 upper=1.57080 effort=10.0 velocity=1.0
