Commit message: real time gazebo physics working

File: src/the_8th_leg_description/urdf/the_8th_leg.urdf.xacro (robot description, xacro)
@@ -17,4 +17,7 @@
     <xacro:property name="link7_wristYawRadius" value="0.025"/>
     <xacro:property name="simplifiedMass" value="1"/>
+    <xacro:property name="joint_effort"   value="50.0"/>
+    <xacro:property name="joint_velocity" value="1.0"/>
+    <xacro:property name="joint_damping"  value="0.5"/>
     <!-- Colors so you can actually see the joints rotate -->
     <material name="grey">
@@ -73,5 +76,6 @@
         <origin xyz="0 0 ${link1_baseLength}"/>
         <axis xyz="0 0 1"/>
-        <limit lower="${-pi}" upper="${pi}" effort="10.0" velocity="1.0"/>
+        <limit lower="${-pi}" upper="${pi}" effort="${joint_effort}" velocity="${joint_velocity}"/>
+        <dynamics damping="${joint_damping}" friction="0.0"/>
     </joint>
     <!-- JOINT 2 : Shoulder pitch, + tips forward toward +X -->
@@ -81,5 +85,6 @@
         <origin xyz="0 0 ${link2_shoulderLength}"/>
         <axis xyz="0 1 0"/>
-        <limit lower="${radians(-108)}" upper="${radians(114)}" effort="10.0" velocity="1.0"/>
+        <limit lower="${radians(-108)}" upper="${radians(114)}" effort="${joint_effort}" velocity="${joint_velocity}"/>
+        <dynamics damping="${joint_damping}" friction="0.0"/>
     </joint>
     <!-- JOINT 3 : Elbow pitch, + folds forward toward +X -->
@@ -89,5 +94,6 @@
         <origin xyz="0 0 ${link3_upperArmLength}"/>
         <axis xyz="0 1 0"/>
-        <limit lower="${radians(-33)}" upper="${radians(150)}" effort="10.0" velocity="1.0"/>
+        <limit lower="${radians(-33)}" upper="${radians(150)}" effort="${joint_effort}" velocity="${joint_velocity}"/>
+        <dynamics damping="${joint_damping}" friction="0.0"/>
     </joint>
     <!-- JOINT 4 : Wrist pitch, + tips forward toward +X -->
@@ -97,5 +103,6 @@
         <origin xyz="0 0 ${link4_lowerArmLength}"/>
         <axis xyz="0 1 0"/>
-        <limit lower="${radians(-100)}" upper="${radians(123)}" effort="10.0" velocity="1.0"/>
+        <limit lower="${radians(-100)}" upper="${radians(123)}" effort="${joint_effort}" velocity="${joint_velocity}"/>
+        <dynamics damping="${joint_damping}" friction="0.0"/>
     </joint>
     <!-- JOINT 5 : Wrist roll, spins about its own long axis (full rotation ok) -->
@@ -105,5 +112,6 @@
         <origin xyz="0 0 ${link5_wristPitchLength}"/>
         <axis xyz="0 0 1"/>
-        <limit lower="${-pi}" upper="${pi}" effort="10.0" velocity="1.0"/>
+        <limit lower="${-pi}" upper="${pi}" effort="${joint_effort}" velocity="${joint_velocity}"/>
+        <dynamics damping="${joint_damping}" friction="0.0"/>
     </joint>
     <!-- JOINT 6 : Wrist yaw. X-axis bend, perpendicular to wrist pitch in the tool frame.
@@ -114,5 +122,6 @@
         <origin xyz="0 0 ${link6_wristRollLength}"/>
         <axis xyz="1 0 0"/>
-        <limit lower="${radians(-90)}" upper="${radians(90)}" effort="10.0" velocity="1.0"/>
+        <limit lower="${radians(-90)}" upper="${radians(90)}" effort="${joint_effort}" velocity="${joint_velocity}"/>
+        <dynamics damping="${joint_damping}" friction="0.0"/>
     </joint>
 </robot>

Commit message: ros2control + joint trajectory controller

File: src/the_8th_leg_description/urdf/the_8th_leg.urdf.xacro (robot description, xacro)
@@ -1,4 +1,5 @@
 <?xml version="1.0"?>
 <robot name="the_8th_leg" xmlns:xacro="http://www.ros.org/wiki/xacro">
+    <xacro:arg name="hardware_plugin" default="gz_ros2_control/GazeboSimSystem"/>
     <!-- Properties -->
     <xacro:property name="link1_baseLength" value="0.02"/>
@@ -125,3 +126,30 @@
         <dynamics damping="${joint_damping}" friction="0.0"/>
     </joint>
+    <!-- ros2_control: interfaces per joint -->
+    <xacro:macro name="joint_ifaces" params="name initial">
+        <joint name="${name}">
+            <command_interface name="position"/>
+            <state_interface name="position">
+                <param name="initial_value">${initial}</param>
+            </state_interface>
+            <state_interface name="velocity"/>
+        </joint>
+    </xacro:macro>
+    <ros2_control name="the_8th_leg_system" type="system">
+        <hardware>
+            <plugin>$(arg hardware_plugin)</plugin>
+        </hardware>
+        <xacro:joint_ifaces name="base_yaw_joint"       initial="0.0"/>
+        <xacro:joint_ifaces name="shoulder_pitch_joint" initial="0.4"/>
+        <xacro:joint_ifaces name="elbow_pitch_joint"    initial="1.0"/>
+        <xacro:joint_ifaces name="wrist_pitch_joint"    initial="0.6"/>
+        <xacro:joint_ifaces name="wrist_roll_joint"     initial="0.0"/>
+        <xacro:joint_ifaces name="wrist_yaw_joint"      initial="0.0"/>
+    </ros2_control>
+    <!-- Gazebo loads ros2_control and starts the controller manager -->
+    <gazebo>
+        <plugin filename="gz_ros2_control-system" name="gz_ros2_control::GazeboSimROS2ControlPlugin">
+            <parameters>$(find the_8th_leg_bringup)/config/controllers.yaml</parameters>
+        </plugin>
+    </gazebo>
 </robot>
